Commit message: finished part F

File: body.urdf (robot description, URDF)
Before this commit: robot robot, 3 links, 2 joints
Joints:
- joint Torso_BackLeg: origin xyz=0.5 0 1 rpy=0 0 0 -> xyz=-0.5 0 1 rpy=0 0 0
- joint Torso_FrontLeg: origin xyz=-0.5 0 1 rpy=0 0 0 -> xyz=0.5 0 1 rpy=0 0 0

Commit message: finished quadruped

File: body.urdf (robot description, URDF)
Before this commit: robot robot, 3 links, 2 joints
Links:
- added link LeftLeg, mass 1; collision box size=1 0.2 0.2; visual box size=1 0.2 0.2
- added link LowerBackLeg, mass 1; collision box size=0.2 0.2 1; visual box size=0.2 0.2 1
- added link LowerFrontLeg, mass 1; collision box size=0.2 0.2 1; visual box size=0.2 0.2 1
- added link LowerLeftLeg, mass 1; collision box size=0.2 0.2 1; visual box size=0.2 0.2 1
- added link LowerRightLeg, mass 1; collision box size=0.2 0.2 1; visual box size=0.2 0.2 1
- added link RightLeg, mass 1; collision box size=1 0.2 0.2; visual box size=1 0.2 0.2
- link BackLeg: geometry collision box size=0.2 1 0.2; visual box size=0.2 1 0.2
- link FrontLeg: geometry collision box size=0.2 1 0.2; visual box size=0.2 1 0.2
Joints:
- added joint BackLeg_LowerBackLeg: type revolute, parent BackLeg, child LowerBackLeg, origin xyz=0 -1 0 rpy=0 0 0, axis 1 0 0, limit lower=-3.14159 upper=3.14159 effort=0.0 velocity=0.0
- added joint FrontLeg_LowerFrontLeg: type revolute, parent FrontLeg, child LowerFrontLeg, origin xyz=0 1 0 rpy=0 0 0, axis 1 0 0, limit lower=-3.14159 upper=3.14159 effort=0.0 velocity=0.0
- added joint LeftLeg_LowerLeftLeg: type revolute, parent LeftLeg, child LowerLeftLeg, origin xyz=1 0 0 rpy=0 0 0, axis 0 1 0, limit lower=-3.14159 upper=3.14159 effort=0.0 velocity=0.0
- added joint Right_LowerRightLeg: type revolute, parent RightLeg, child LowerRightLeg, origin xyz=-1 0 0 rpy=0 0 0, axis 0 1 0, limit lower=-3.14159 upper=3.14159 effort=0.0 velocity=0.0
- added joint Torso_LeftLeg: type revolute, parent Torso, child LeftLeg, origin xyz=0.5 0 1 rpy=0 0 0, axis 0 1 0, limit lower=-3.14159 upper=3.14159 effort=0.0 velocity=0.0
- added joint Torso_RightLeg: type revolute, parent Torso, child RightLeg, origin xyz=-0.5 0 1 rpy=0 0 0, axis 0 1 0, limit lower=-3.14159 upper=3.14159 effort=0.0 velocity=0.0
- joint Torso_BackLeg: axis 0 1 0 -> 1 0 0; origin xyz=-0.5 0 1 rpy=0 0 0 -> xyz=0 -0.5 1 rpy=0 0 0
- joint Torso_FrontLeg: axis 0 1 0 -> 1 0 0; origin xyz=0.5 0 1 rpy=0 0 0 -> xyz=0 0.5 1 rpy=0 0 0

Commit message: finished assignment 5

File: body.urdf (robot description, URDF)
Before this commit: robot robot, 9 links, 8 joints
Links:
- added link BackLegFoot, mass 1; collision box size=0.2 0.2 0.75; visual box size=0.2 0.2 0.75
- added link FrontLegFoot, mass 1; collision box size=0.2 0.2 0.75; visual box size=0.2 0.2 0.75
- added link LeftLegFoot, mass 1; collision box size=0.2 0.2 0.75; visual box size=0.2 0.2 0.75
- added link RightLegFoot, mass 1; collision box size=0.2 0.2 0.75; visual box size=0.2 0.2 0.75
- link BackLeg: geometry collision box size=0.2 0.3 0.2; visual box size=0.2 0.3 0.2
- link FrontLeg: geometry collision box size=0.2 0.3 0.2; visual box size=0.2 0.3 0.2
- link LeftLeg: geometry collision box size=0.2 0.3 0.2; visual box size=0.2 0.3 0.2
- link LowerBackLeg: geometry collision box size=0.5 0.2 0.2; visual box size=0.5 0.2 0.2
- link LowerFrontLeg: geometry collision box size=0.5 0.2 0.2; visual box size=0.5 0.2 0.2
- link LowerLeftLeg: geometry collision box size=0.5 0.2 0.2; visual box size=0.5 0.2 0.2
- link LowerRightLeg: geometry collision box size=0.5 0.2 0.2; visual box size=0.5 0.2 0.2
- link RightLeg: geometry collision box size=0.2 0.3 0.2; visual box size=0.2 0.3 0.2
- link Torso: geometry collision box size=2 0.8 0.6; visual box size=2 0.8 0.6
Joints:
- removed joint Right_LowerRightLeg
- added joint LowerBackLeg_BackLegFoot: type revolute, parent LowerBackLeg, child BackLegFoot, origin xyz=0.2 0 -0.5 rpy=0 0 0, axis 0 1 0, limit lower=-3.14159 upper=3.14159 effort=0.0 velocity=0.0
- added joint LowerFrontLeg_FrontLegFoot: type revolute, parent LowerFrontLeg, child FrontLegFoot, origin xyz=0.2 0 -0.5 rpy=0 0 0, axis 0 1 0, limit lower=-3.14159 upper=3.14159 effort=0.0 velocity=0.0
- added joint LowerLeftLeg_LeftLegFoot: type revolute, parent LowerLeftLeg, child LeftLegFoot, origin xyz=0.2 0 -0.5 rpy=0 0 0, axis 0 1 0, limit lower=-3.14159 upper=3.14159 effort=0.0 velocity=0.0
- added joint LowerRightLeg_RightLegFoot: type revolute, parent LowerRightLeg, child RightLegFoot, origin xyz=0.2 0 -0.5 rpy=0 0 0, axis 0 1 0, limit lower=-3.14159 upper=3.14159 effort=0.0 velocity=0.0
- added joint RightLeg_LowerRightLeg: type revolute, parent RightLeg, child LowerRightLeg, origin xyz=0.2 -0.6 0 rpy=0 0 0, axis 0 1 0, limit lower=-3.14159 upper=3.14159 effort=0.0 velocity=0.0
- joint BackLeg_LowerBackLeg: axis 1 0 0 -> 0 1 0; origin xyz=0 -1 0 rpy=0 0 0 -> xyz=0.2 -0.6 0 rpy=0 0 0
- joint FrontLeg_LowerFrontLeg: axis 1 0 0 -> 0 1 0; origin xyz=0 1 0 rpy=0 0 0 -> xyz=0.2 0.6 0 rpy=0 0 0
- joint LeftLeg_LowerLeftLeg: origin xyz=1 0 0 rpy=0 0 0 -> xyz=0.2 0.6 0 rpy=0 0 0
- joint Torso_BackLeg: axis 1 0 0 -> 0 1 0; origin xyz=0 -0.5 1 rpy=0 0 0 -> xyz=-0.8 -0.1 1 rpy=0 0 0
- joint Torso_FrontLeg: axis 1 0 0 -> 0 1 0; origin xyz=0 0.5 1 rpy=0 0 0 -> xyz=-0.8 0.1 1 rpy=0 0 0
- joint Torso_LeftLeg: origin xyz=0.5 0 1 rpy=0 0 0 -> xyz=0.8 0.1 1 rpy=0 0 0
- joint Torso_RightLeg: origin xyz=-0.5 0 1 rpy=0 0 0 -> xyz=0.8 -0.1 1 rpy=0 0 0

Commit message: finished assignment 6

File: body.urdf (robot description, URDF)
Before this commit: robot robot, 13 links, 12 joints
Links:
- removed link BackLeg
- removed link BackLegFoot
- removed link FrontLeg
- removed link FrontLegFoot
- removed link LeftLeg
- removed link LeftLegFoot
- removed link LowerBackLeg
- removed link LowerFrontLeg
- removed link LowerLeftLeg
- removed link LowerRightLeg
- removed link RightLeg
- removed link RightLegFoot
- removed link Torso
- added link Cube0, mass 1; collision box size=1.2 2.6 2.4; visual box size=1.2 2.6 2.4
- added link Cube1, mass 1; collision box size=2.6 2.4 2.4; visual box size=2.6 2.4 2.4
- added link Cube2, mass 1; collision box size=1.2 2.6 3.0; visual box size=1.2 2.6 3.0
- added link Cube3, mass 1; collision box size=1.2 1.8 1.6; visual box size=1.2 1.8 1.6
- added link Cube4, mass 1; collision box size=1.2 2.6 2.6; visual box size=1.2 2.6 2.6
- added link Cube5, mass 1; collision box size=2.0 3.0 3.0; visual box size=2.0 3.0 3.0
Joints:
- removed joint BackLeg_LowerBackLeg
- removed joint FrontLeg_LowerFrontLeg
- removed joint LeftLeg_LowerLeftLeg
- removed joint LowerBackLeg_BackLegFoot
- removed joint LowerFrontLeg_FrontLegFoot
- removed joint LowerLeftLeg_LeftLegFoot
- removed joint LowerRightLeg_RightLegFoot
- removed joint RightLeg_LowerRightLeg
- removed joint Torso_BackLeg
- removed joint Torso_FrontLeg
- removed joint Torso_LeftLeg
- removed joint Torso_RightLeg
- added joint Cube0_Cube1: type revolute, parent Cube0, child Cube1, origin xyz=0 1.3 0 rpy=0 0 0, axis 1 0 0, limit lower=-3.14159 upper=3.14159 effort=0.0 velocity=0.0
- added joint Cube1_Cube2: type revolute, parent Cube1, child Cube2, origin xyz=0 2.4 0 rpy=0 0 0, axis 1 0 0, limit lower=-3.14159 upper=3.14159 effort=0.0 velocity=0.0
- added joint Cube2_Cube3: type revolute, parent Cube2, child Cube3, origin xyz=0 2.6 0 rpy=0 0 0, axis 1 0 0, limit lower=-3.14159 upper=3.14159 effort=0.0 velocity=0.0
- added joint Cube3_Cube4: type revolute, parent Cube3, child Cube4, origin xyz=0 1.8 0 rpy=0 0 0, axis 1 0 0, limit lower=-3.14159 upper=3.14159 effort=0.0 velocity=0.0
- added joint Cube4_Cube5: type revolute, parent Cube4, child Cube5, origin xyz=0 2.6 0 rpy=0 0 0, axis 1 0 0, limit lower=-3.14159 upper=3.14159 effort=0.0 velocity=0.0

Commit message: start of 7

File: body.urdf (robot description, URDF)
Before this commit: robot robot, 6 links, 5 joints
Links:
- added link Cube6, mass 1; collision box size=0.7727947880941977 1.1825358898406702 1.0573853315511754; visual box size=0.7727947880941977 1.1825358898406702 1.0573853315511754
- added link Cube7, mass 1; collision box size=1.1146218885423036 1.4228518478201826 1.3188469511711094; visual box size=1.1146218885423036 1.4228518478201826 1.3188469511711094
- link Cube0: geometry collision box size=1.2061091339124892 1.1681133373044195 0.6117615489816307; visual box size=1.2061091339124892 1.1681133373044195 0.6117615489816307
- link Cube1: geometry collision box size=0.5504521719972292 1.0360730580366457 0.9223179336096364; visual box size=0.5504521719972292 1.0360730580366457 0.9223179336096364
- link Cube2: geometry collision box size=0.7297897198399328 1.2450221332714992 1.3625506835184455; visual box size=0.7297897198399328 1.2450221332714992 1.3625506835184455
- link Cube3: geometry collision box size=1.4599033381265536 1.2801248341404778 1.0034428448791073; visual box size=1.4599033381265536 1.2801248341404778 1.0034428448791073
- link Cube4: geometry collision box size=1.1090060144054719 1.316839192033532 1.443961905555287; visual box size=1.1090060144054719 1.316839192033532 1.443961905555287
- link Cube5: geometry collision box size=1.3735136643540637 0.6115795554415795 0.5857717564878926; visual box size=1.3735136643540637 0.6115795554415795 0.5857717564878926
Joints:
- removed joint Cube2_Cube3
- removed joint Cube3_Cube4
- removed joint Cube4_Cube5
- added joint Cube0_Cube4: type revolute, parent Cube0, child Cube4, origin xyz=-1.2061091339124892 0 0 rpy=0 0 0, axis 1 0 0, limit lower=-3.14159 upper=3.14159 effort=0.0 velocity=0.0
- added joint Cube1_Cube3: type revolute, parent Cube1, child Cube3, origin xyz=-0.5504521719972292 0 0 rpy=0 0 0, axis 1 0 0, limit lower=-3.14159 upper=3.14159 effort=0.0 velocity=0.0
- added joint Cube1_Cube5: type revolute, parent Cube1, child Cube5, origin xyz=-0.5504521719972292 0 0 rpy=0 0 0, axis 1 0 0, limit lower=-3.14159 upper=3.14159 effort=0.0 velocity=0.0
- added joint Cube2_Cube6: type revolute, parent Cube2, child Cube6, origin xyz=0 0 -1.3625506835184455 rpy=0 0 0, axis 1 0 0, limit lower=-3.14159 upper=3.14159 effort=0.0 velocity=0.0
- added joint Cube6_Cube7: type revolute, parent Cube6, child Cube7, origin xyz=0 1.1825358898406702 0 rpy=0 0 0, axis 1 0 0, limit lower=-3.14159 upper=3.14159 effort=0.0 velocity=0.0
- joint Cube0_Cube1: origin xyz=0 1.3 0 rpy=0 0 0 -> xyz=1.2061091339124892 0 0 rpy=0 0 0
- joint Cube1_Cube2: origin xyz=0 2.4 0 rpy=0 0 0 -> xyz=0 0 -0.9223179336096364 rpy=0 0 0

Commit message: finished assignment 7

File: body.urdf (robot description, URDF)
Before this commit: robot robot, 8 links, 7 joints
Links:
- removed link Cube7
- link Cube0: geometry collision box size=1.2273821388761017 1.0677780656362548 0.8542440863595545; visual box size=1.2273821388761017 1.0677780656362548 0.8542440863595545
- link Cube1: geometry collision box size=0.6078500277440819 1.407118169673336 0.5847232950220143; visual box size=0.6078500277440819 1.407118169673336 0.5847232950220143
- link Cube2: geometry collision box size=1.132454104937534 0.5021736237319693 1.0575636406475568; visual box size=1.132454104937534 0.5021736237319693 1.0575636406475568
- link Cube3: geometry collision box size=0.9134831481567219 0.8475281094460102 1.020857810997415; visual box size=0.9134831481567219 0.8475281094460102 1.020857810997415
- link Cube4: geometry collision box size=1.3639849403921067 0.953491941370818 1.2861275480575456; visual box size=1.3639849403921067 0.953491941370818 1.2861275480575456
- link Cube5: geometry collision box size=1.132855008560607 0.6907908360449134 1.0333179048110601; visual box size=1.132855008560607 0.6907908360449134 1.0333179048110601
- link Cube6: geometry collision box size=1.0899031214099404 0.960797254468928 0.8234640438461336; visual box size=1.0899031214099404 0.960797254468928 0.8234640438461336
Joints:
- removed joint Cube0_Cube4
- removed joint Cube1_Cube3
- removed joint Cube1_Cube5
- removed joint Cube2_Cube6
- removed joint Cube6_Cube7
- added joint Cube2_Cube3: type revolute, parent Cube2, child Cube3, origin xyz=-1.132454104937534 0 0 rpy=0 0 0, axis 1 0 0, limit lower=-3.14159 upper=3.14159 effort=0.0 velocity=0.0
- added joint Cube3_Cube4: type revolute, parent Cube3, child Cube4, origin xyz=-0.9134831481567219 0 0 rpy=0 0 0, axis 1 0 0, limit lower=-3.14159 upper=3.14159 effort=0.0 velocity=0.0
- added joint Cube4_Cube5: type revolute, parent Cube4, child Cube5, origin xyz=0 0 1.2861275480575456 rpy=0 0 0, axis 1 0 0, limit lower=-3.14159 upper=3.14159 effort=0.0 velocity=0.0
- added joint Cube5_Cube6: type revolute, parent Cube5, child Cube6, origin xyz=0 -0.6907908360449134 0 rpy=0 0 0, axis 1 0 0, limit lower=-3.14159 upper=3.14159 effort=0.0 velocity=0.0
- joint Cube0_Cube1: origin xyz=1.2061091339124892 0 0 rpy=0 0 0 -> xyz=0 -1.0677780656362548 0 rpy=0 0 0
- joint Cube1_Cube2: origin xyz=0 0 -0.9223179336096364 rpy=0 0 0 -> xyz=0 -1.407118169673336 0 rpy=0 0 0

Commit message: finished assignment7

File: body.urdf (robot description, URDF)
Before this commit: robot robot, 7 links, 6 joints
Links:
- removed link Cube6
- link Cube0: geometry collision box size=0.84904386910402 0.6616318779042362 1.2683370509140222; visual box size=0.84904386910402 0.6616318779042362 1.2683370509140222
- link Cube1: geometry collision box size=0.6300411485268356 0.8742147199097677 1.2515844317932046; visual box size=0.6300411485268356 0.8742147199097677 1.2515844317932046
- link Cube2: geometry collision box size=0.5962410535917851 1.1560291499627384 1.254440425420498; visual box size=0.5962410535917851 1.1560291499627384 1.254440425420498
- link Cube3: geometry collision box size=1.0442304906746438 0.8084203044039545 1.3801180749405597; visual box size=1.0442304906746438 0.8084203044039545 1.3801180749405597
- link Cube4: geometry collision box size=1.0446107970413472 0.6234655258229708 0.6288965528947907; visual box size=1.0446107970413472 0.6234655258229708 0.6288965528947907
- link Cube5: geometry collision box size=0.8860765068346297 0.8898322427158593 1.331603534130965; visual box size=0.8860765068346297 0.8898322427158593 1.331603534130965
Joints:
- removed joint Cube1_Cube2
- removed joint Cube2_Cube3
- removed joint Cube3_Cube4
- removed joint Cube4_Cube5
- removed joint Cube5_Cube6
- added joint Cube0_Cube2: type revolute, parent Cube0, child Cube2, origin xyz=-0.0 -0.0 1.254440425420498 rpy=0 0 0, axis 1 0 0, limit lower=-3.14159 upper=3.14159 effort=0.0 velocity=0.0
- added joint Cube0_Cube4: type revolute, parent Cube0, child Cube4, origin xyz=-0.0 -0.0 -0.6288965528947907 rpy=0 0 0, axis 1 0 0, limit lower=-3.14159 upper=3.14159 effort=0.0 velocity=0.0
- added joint Cube0_Cube5: type revolute, parent Cube0, child Cube5, origin xyz=-0.8860765068346297 -0.0 -0.0 rpy=0 0 0, axis 1 0 0, limit lower=-3.14159 upper=3.14159 effort=0.0 velocity=0.0
- added joint Cube1_Cube3: type revolute, parent Cube1, child Cube3, origin xyz=-0.0 -0.0 -1.3801180749405597 rpy=0 0 0, axis 1 0 0, limit lower=-3.14159 upper=3.14159 effort=0.0 velocity=0.0
- joint Cube0_Cube1: origin xyz=0 -1.0677780656362548 0 rpy=0 0 0 -> xyz=-0.0 -0.8742147199097677 -0.0 rpy=0 0 0

Commit message: finishied assignment 8

File: body.urdf (robot description, URDF)
Before this commit: robot robot, 6 links, 5 joints
Links:
- added link Cube10, mass 1; collision box size=0.24245806451509322 0.3114868426561775 0.2; visual box size=0.24245806451509322 0.3114868426561775 0.2
- added link Cube11, mass 1; collision box size=0.47933765909542886 0.2 0.2; visual box size=0.47933765909542886 0.2 0.2
- added link Cube12, mass 1; collision box size=0.2 0.2 0.75; visual box size=0.2 0.2 0.75
- added link Cube6, mass 1; collision box size=0.2 0.2 0.75; visual box size=0.2 0.2 0.75
- added link Cube7, mass 1; collision box size=0.2 0.3 0.2; visual box size=0.2 0.3 0.2
- added link Cube8, mass 1; collision box size=0.5 0.2 0.2; visual box size=0.5 0.2 0.2
- added link Cube9, mass 1; collision box size=0.2 0.2 0.75; visual box size=0.2 0.2 0.75
- link Cube0: geometry collision box size=1.9664980389513627 0.8 0.6; visual box size=1.9664980389513627 0.8 0.6
- link Cube1: geometry collision box size=0.2 0.3 0.2; visual box size=0.2 0.3 0.2
- link Cube2: geometry collision box size=0.5 0.2 0.2; visual box size=0.5 0.2 0.2
- link Cube3: geometry collision box size=0.2 0.19498957428757396 0.75; visual box size=0.2 0.19498957428757396 0.75
- link Cube4: geometry collision box size=0.1930262358437866 0.3 0.2; visual box size=0.1930262358437866 0.3 0.2
- link Cube5: geometry collision box size=0.5 0.2 0.2; visual box size=0.5 0.2 0.2
Joints:
- removed joint Cube0_Cube2
- removed joint Cube0_Cube5
- removed joint Cube1_Cube3
- added joint Cube0_Cube10: type revolute, parent Cube0, child Cube10, origin xyz=0.32 0.09999999999999999 1 rpy=0 0 0, axis 0 1 0, limit lower=-3.14159 upper=3.14159 effort=0.0 velocity=0.0
- added joint Cube0_Cube7: type revolute, parent Cube0, child Cube7, origin xyz=0.32 -0.09999999999999999 1 rpy=0 0 0, axis 0 1 0, limit lower=-3.14159 upper=3.14159 effort=0.0 velocity=0.0
- added joint Cube10_Cube11: type revolute, parent Cube10, child Cube11, origin xyz=0.24245806451509322 -0.622973685312355 0 rpy=0 0 0, axis 0 1 0, limit lower=-3.14159 upper=3.14159 effort=0.0 velocity=0.0
- added joint Cube11_Cube12: type revolute, parent Cube11, child Cube12, origin xyz=0.15977921969847628 0 -0.5 rpy=0 0 0, axis 0 1 0, limit lower=-3.14159 upper=3.14159 effort=0.0 velocity=0.0
- added joint Cube1_Cube2: type revolute, parent Cube1, child Cube2, origin xyz=0.2 0.6 0 rpy=0 0 0, axis 0 1 0, limit lower=-3.14159 upper=3.14159 effort=0.0 velocity=0.0
- added joint Cube2_Cube3: type revolute, parent Cube2, child Cube3, origin xyz=0.16666666666666666 0 -0.5 rpy=0 0 0, axis 0 1 0, limit lower=-3.14159 upper=3.14159 effort=0.0 velocity=0.0
- added joint Cube4_Cube5: type revolute, parent Cube4, child Cube5, origin xyz=0.1930262358437866 -0.6 0 rpy=0 0 0, axis 0 1 0, limit lower=-3.14159 upper=3.14159 effort=0.0 velocity=0.0
- added joint Cube5_Cube6: type revolute, parent Cube5, child Cube6, origin xyz=0.16666666666666666 0 -0.5 rpy=0 0 0, axis 0 1 0, limit lower=-3.14159 upper=3.14159 effort=0.0 velocity=0.0
- added joint Cube7_Cube8: type revolute, parent Cube7, child Cube8, origin xyz=0.2 0.6 0 rpy=0 0 0, axis 0 1 0, limit lower=-3.14159 upper=3.14159 effort=0.0 velocity=0.0
- added joint Cube8_Cube9: type revolute, parent Cube8, child Cube9, origin xyz=0.16666666666666666 0 -0.5 rpy=0 0 0, axis 0 1 0, limit lower=-3.14159 upper=3.14159 effort=0.0 velocity=0.0
- joint Cube0_Cube1: axis 1 0 0 -> 0 1 0; origin xyz=-0.0 -0.8742147199097677 -0.0 rpy=0 0 0 -> xyz=-0.32 0.09999999999999999 1 rpy=0 0 0
- joint Cube0_Cube4: axis 1 0 0 -> 0 1 0; origin xyz=-0.0 -0.0 -0.6288965528947907 rpy=0 0 0 -> xyz=-0.32 -0.09999999999999999 1 rpy=0 0 0

Commit message: made simulation run better

File: body.urdf (robot description, URDF)
Before this commit: robot robot, 13 links, 12 joints
Links:
- link Cube0: geometry collision box size=2.0079880312205423 0.7873933286567052 0.5930763529476415; visual box size=2.0079880312205423 0.7873933286567052 0.5930763529476415
- link Cube1: geometry collision box size=0.19520347268119181 0.3217037277888413 0.15157168024405965; visual box size=0.19520347268119181 0.3217037277888413 0.15157168024405965
- link Cube10: geometry collision box size=0.205969993499582 0.2616423250481231 0.2208252471599626; visual box size=0.205969993499582 0.2616423250481231 0.2208252471599626
- link Cube11: geometry collision box size=0.5048879534625015 0.20712298888986802 0.1997421107044769; visual box size=0.5048879534625015 0.20712298888986802 0.1997421107044769
- link Cube12: geometry collision box size=0.24733100198371039 0.17056400500288443 0.7081432439738179; visual box size=0.24733100198371039 0.17056400500288443 0.7081432439738179
- link Cube2: geometry collision box size=0.47076664870371127 0.2357242257954038 0.1519394961332025; visual box size=0.47076664870371127 0.2357242257954038 0.1519394961332025
- link Cube3: geometry collision box size=0.24281226748139123 0.17868569558749864 0.7587902191974266; visual box size=0.24281226748139123 0.17868569558749864 0.7587902191974266
- link Cube4: geometry collision box size=0.20447743786280348 0.28820902249848407 0.1633495874569597; visual box size=0.20447743786280348 0.28820902249848407 0.1633495874569597
- link Cube5: geometry collision box size=0.4816858807144658 0.153353381191003 0.1686602644336262; visual box size=0.4816858807144658 0.153353381191003 0.1686602644336262
- link Cube6: geometry collision box size=0.24068558705020804 0.23643969419612354 0.756070503718337; visual box size=0.24068558705020804 0.23643969419612354 0.756070503718337
- link Cube7: geometry collision box size=0.20871697428972824 0.29357469153295085 0.23885281952397475; visual box size=0.20871697428972824 0.29357469153295085 0.23885281952397475
- link Cube8: geometry collision box size=0.5437352451708659 0.17540978705713642 0.1617302597459337; visual box size=0.5437352451708659 0.17540978705713642 0.1617302597459337
- link Cube9: geometry collision box size=0.1544113994859459 0.1762358609516454 0.7001262620022505; visual box size=0.1544113994859459 0.1762358609516454 0.7001262620022505
Joints:
- joint Cube0_Cube1: origin xyz=-0.32 0.09999999999999999 1 rpy=0 0 0 -> xyz=-0.31495733146268207 0.10723457592961377 1 rpy=0 0 0
- joint Cube0_Cube10: origin xyz=0.32 0.09999999999999999 1 rpy=0 0 0 -> xyz=0.31495733146268207 0.09606967416616136 1 rpy=0 0 0
- joint Cube0_Cube4: origin xyz=-0.32 -0.09999999999999999 1 rpy=0 0 0 -> xyz=-0.31495733146268207 -0.09606967416616136 1 rpy=0 0 0
- joint Cube0_Cube7: origin xyz=0.32 -0.09999999999999999 1 rpy=0 0 0 -> xyz=0.31495733146268207 -0.09606967416616136 1 rpy=0 0 0
- joint Cube10_Cube11: origin xyz=0.24245806451509322 -0.622973685312355 0 rpy=0 0 0 -> xyz=0.205969993499582 -0.5232846500962463 0 rpy=0 0 0
- joint Cube11_Cube12: origin xyz=0.15977921969847628 0 -0.5 rpy=0 0 0 -> xyz=0.12622198836562537 0 -0.5 rpy=0 0 0
- joint Cube1_Cube2: origin xyz=0.2 0.6 0 rpy=0 0 0 -> xyz=0.19520347268119181 0.6434074555776826 0 rpy=0 0 0
- joint Cube2_Cube3: origin xyz=0.16666666666666666 0 -0.5 rpy=0 0 0 -> xyz=0.11769166217592782 0 -0.5 rpy=0 0 0
- joint Cube4_Cube5: origin xyz=0.1930262358437866 -0.6 0 rpy=0 0 0 -> xyz=0.20447743786280348 -0.5764180449969681 0 rpy=0 0 0
- joint Cube5_Cube6: origin xyz=0.16666666666666666 0 -0.5 rpy=0 0 0 -> xyz=0.12042147017861644 0 -0.5 rpy=0 0 0
- joint Cube7_Cube8: origin xyz=0.2 0.6 0 rpy=0 0 0 -> xyz=0.20871697428972824 0.5871493830659017 0 rpy=0 0 0
- joint Cube8_Cube9: origin xyz=0.16666666666666666 0 -0.5 rpy=0 0 0 -> xyz=0.13593381129271648 0 -0.5 rpy=0 0 0
