Commit message: finished readme

File: body.urdf (robot description, URDF)
Before this commit: robot robot, 13 links, 12 joints
Links:
- link Cube0: geometry collision box size=2.0481756641186633 0.8393021212196285 0.6259348794956328; visual box size=2.0481756641186633 0.8393021212196285 0.6259348794956328
- link Cube1: geometry collision box size=0.21511205589027865 0.25396835020657266 0.23138763651723376; visual box size=0.21511205589027865 0.25396835020657266 0.23138763651723376
- link Cube10: geometry collision box size=0.20227366296364224 0.3236811465828239 0.166540611484626; visual box size=0.20227366296364224 0.3236811465828239 0.166540611484626
- link Cube11: geometry collision box size=0.5187058292433259 0.1926810840028242 0.22285573975501832; visual box size=0.5187058292433259 0.1926810840028242 0.22285573975501832
- link Cube12: geometry collision box size=0.22563353922144797 0.18976112823946484 0.7925200108860829; visual box size=0.22563353922144797 0.18976112823946484 0.7925200108860829
- link Cube2: geometry collision box size=0.5262573134667063 0.19552824669879854 0.2031826451335968; visual box size=0.5262573134667063 0.19552824669879854 0.2031826451335968
- link Cube3: geometry collision box size=0.16093360675852392 0.1646032745988229 0.7508788738779337; visual box size=0.16093360675852392 0.1646032745988229 0.7508788738779337
- link Cube4: geometry collision box size=0.17156502809027913 0.38932028521254297 0.19621525128552286; visual box size=0.17156502809027913 0.38932028521254297 0.19621525128552286
- link Cube5: geometry collision box size=0.4632267274456731 0.22642416087544281 0.1712733698112648; visual box size=0.4632267274456731 0.22642416087544281 0.1712733698112648
- link Cube6: geometry collision box size=0.15742584333581777 0.15549645327085687 0.7162205510337177; visual box size=0.15742584333581777 0.15549645327085687 0.7162205510337177
- link Cube7: geometry collision box size=0.18564636801206702 0.2595307810639996 0.1643263006161409; visual box size=0.18564636801206702 0.2595307810639996 0.1643263006161409
- link Cube8: geometry collision box size=0.5431012933250224 0.20765842163910742 0.23396452138186097; visual box size=0.5431012933250224 0.20765842163910742 0.23396452138186097
- link Cube9: geometry collision box size=0.21232921128220617 0.18245174964216432 0.7728011643402769; visual box size=0.21232921128220617 0.18245174964216432 0.7728011643402769
Joints:
- joint Cube0_Cube1: origin xyz=-0.31495733146268207 0.10723457592961377 1 rpy=0 0 0 -> xyz=-0.33572084848785144 0.08465611673552421 1 rpy=0 0 0
- joint Cube0_Cube10: origin xyz=0.31495733146268207 0.09606967416616136 1 rpy=0 0 0 -> xyz=0.33572084848785144 0.129773428404181 1 rpy=0 0 0
- joint Cube0_Cube4: origin xyz=-0.31495733146268207 -0.09606967416616136 1 rpy=0 0 0 -> xyz=-0.33572084848785144 -0.129773428404181 1 rpy=0 0 0
- joint Cube0_Cube7: origin xyz=0.31495733146268207 -0.09606967416616136 1 rpy=0 0 0 -> xyz=0.33572084848785144 -0.129773428404181 1 rpy=0 0 0
- joint Cube10_Cube11: origin xyz=0.205969993499582 -0.5232846500962463 0 rpy=0 0 0 -> xyz=0.20227366296364224 -0.6473622931656478 0 rpy=0 0 0
- joint Cube11_Cube12: origin xyz=0.12622198836562537 0 -0.5 rpy=0 0 0 -> xyz=0.12967645731083147 0 -0.5 rpy=0 0 0
- joint Cube1_Cube2: origin xyz=0.19520347268119181 0.6434074555776826 0 rpy=0 0 0 -> xyz=0.21511205589027865 0.5079367004131453 0 rpy=0 0 0
- joint Cube2_Cube3: origin xyz=0.11769166217592782 0 -0.5 rpy=0 0 0 -> xyz=0.1315643283666766 0 -0.5 rpy=0 0 0
- joint Cube4_Cube5: origin xyz=0.20447743786280348 -0.5764180449969681 0 rpy=0 0 0 -> xyz=0.17156502809027913 -0.7786405704250859 0 rpy=0 0 0
- joint Cube5_Cube6: origin xyz=0.12042147017861644 0 -0.5 rpy=0 0 0 -> xyz=0.11580668186141828 0 -0.5 rpy=0 0 0
- joint Cube7_Cube8: origin xyz=0.20871697428972824 0.5871493830659017 0 rpy=0 0 0 -> xyz=0.18564636801206702 0.5190615621279993 0 rpy=0 0 0
- joint Cube8_Cube9: origin xyz=0.13593381129271648 0 -0.5 rpy=0 0 0 -> xyz=0.1357753233312556 0 -0.5 rpy=0 0 0
